File: LEDBeam.sch (KiCad schematic (older format))
At the start: 12 parts, among them J1 Power, J2 Switch, J3 Power led, U1 WeMos_D1_mini, U2 LED_Dimmer_Platine, U3 LED_Dimmer_Platine, U4 LM7805_TO220, U5 LED_Dimmer_Platine, U6 LED_Dimmer_Platine

Commit message: New board design
Parts:
- U2, U3, U5, U6: footprint Connector_PinHeader_2.54mm:PinHeader_1x07_P2.54mm_Vertical -> LEDBeam:LED_Driver_module
Connections:
- net B_PWM: now also U1.4 (SCK/D5); no longer U1.5 (MISO/D6)
- net W_PWM: now also U1.5 (MISO/D6); no longer U1.4 (SCK/D5)
- net 24V renamed +24V
- net 5V renamed +5V
